File: mainboard2026_0522/mainboard2026_0522.kicad_pcb (KiCad board)
At the start: 2 copper layers, 0 parts

Commit message: pcb_precomplete
Parts:
- added 10k1: R, Resistor_SMD:R_0603_1608Metric_Pad0.98x0.95mm_HandSolder, B.Cu at (151.0, 45.0)
- added C1: 0.1u, Capacitor_SMD:C_0603_1608Metric_Pad1.08x0.95mm_HandSolder, F.Cu at (166.0, 78.0)
- added C10: 0.1u, Capacitor_SMD:C_0603_1608Metric_Pad1.08x0.95mm_HandSolder, B.Cu at (146.0, 45.0)
- added C11: 0.1u, Capacitor_SMD:C_0603_1608Metric_Pad1.08x0.95mm_HandSolder, B.Cu at (123.5, 51.0)
- added C12: 4.7u, Capacitor_SMD:C_0603_1608Metric_Pad1.08x0.95mm_HandSolder, B.Cu at (79.5, 55.0)
- added C13: 0.1u, Capacitor_SMD:C_0603_1608Metric_Pad1.08x0.95mm_HandSolder, B.Cu at (84.6, 55.0)
- added C2: 0.1u, Capacitor_SMD:C_0603_1608Metric_Pad1.08x0.95mm_HandSolder, F.Cu at (170.5, 78.0)
- added C3: 0.1u, Capacitor_SMD:C_0603_1608Metric_Pad1.08x0.95mm_HandSolder, B.Cu at (201.4, 64.0)
- added C4: 0.1u, Capacitor_SMD:C_0603_1608Metric_Pad1.08x0.95mm_HandSolder, F.Cu at (175.5, 78.0)
- added C9: C_Polarized, Capacitor_THT:CP_Radial_D6.3mm_P2.50mm, F.Cu at (173.8, 60.5)
- added J1: Conn_01x06, Connector_JST:JST_XH_S6B-XH-A-1_1x06_P2.50mm_Horizontal, B.Cu at (110.0, 42.1)
- added J10: Conn_01x06_Pin, Connector_JST:JST_XH_S6B-XH-A-1_1x06_P2.50mm_Horizontal, B.Cu at (187.5, 118.0)
- added J11: Conn_01x02_Pin, Connector_JST:JST_PH_B2B-PH-K_1x02_P2.00mm_Vertical, B.Cu at (158.5, 40.5)
- added J12: Conn_01x02_Pin, Connector_JST:JST_PH_B2B-PH-K_1x02_P2.00mm_Vertical, F.Cu at (167.5, 61.5)
- added J13: Conn_01x02, Connector_AMASS:AMASS_XT30U-M_1x02_P5.0mm_Vertical, B.Cu at (85.0, 42.5)
- added J2: Conn_01x06, Connector_JST:JST_XH_S6B-XH-A-1_1x06_P2.50mm_Horizontal, B.Cu at (177.0, 42.5)
- added J3: Conn_01x02_Pin, Connector_JST:JST_PH_B2B-PH-K_1x02_P2.00mm_Vertical, F.Cu at (168.5, 115.5)
- added J7: Conn_01x02, Connector_PinHeader_2.54mm:PinHeader_1x02_P2.54mm_Vertical, F.Cu at (200.0, 106.5)
- added J8: Conn_01x03_Pin, Connector_JST:JST_PH_B3B-PH-K_1x03_P2.00mm_Vertical, B.Cu at (99.0, 99.0)
- added J9: Conn_01x06_Pin, Connector_JST:JST_XH_S6B-XH-A-1_1x06_P2.50mm_Horizontal, B.Cu at (68.0, 118.5)
- added Q1: Q_NMOS_GDS, Package_TO_SOT_SMD:TO-252-3_TabPin2, F.Cu at (180.2, 116.5)
- added Q2: Q_NMOS_GDS, Package_TO_SOT_SMD:TO-252-3_TabPin2, F.Cu at (172.1, 70.5)
- added R1: 10k, Resistor_SMD:R_0603_1608Metric_Pad0.98x0.95mm_HandSolder, B.Cu at (191.6, 64.0)
- added R12: 10k, Resistor_SMD:R_0603_1608Metric_Pad0.98x0.95mm_HandSolder, F.Cu at (184.1, 72.5)
- added R13: 10k, Resistor_SMD:R_0603_1608Metric_Pad0.98x0.95mm_HandSolder, F.Cu at (184.1, 76.0)
- added R2: 10k, Resistor_SMD:R_0603_1608Metric_Pad0.98x0.95mm_HandSolder, F.Cu at (173.5, 113.5)
- added R3: 10k, Resistor_SMD:R_0603_1608Metric_Pad0.98x0.95mm_HandSolder, F.Cu at (173.5, 118.6)
- added R4: 10k, Resistor_SMD:R_0603_1608Metric_Pad0.98x0.95mm_HandSolder, B.Cu at (116.5, 109.5)
- added R5: 1k, Resistor_SMD:R_0603_1608Metric_Pad0.98x0.95mm_HandSolder, F.Cu at (188.6, 72.5)
- added R6: 10k, Resistor_SMD:R_0603_1608Metric_Pad0.98x0.95mm_HandSolder, B.Cu at (182.1, 64.0)
- added R9: 10k, Resistor_SMD:R_0603_1608Metric_Pad0.98x0.95mm_HandSolder, F.Cu at (188.6, 76.0)
- added SW1: SW_SPDT, Button_Switch_THT:SW_Slide-03_Wuerth-WS-SLTV_10x2.5x6.4_P2.54mm, B.Cu at (148.0, 40.0)
- added SW2: SW_Push, Button_Switch_THT:SW_PUSH_6mm_H7.3mm, B.Cu at (140.5, 40.0)
- added U1: Bno055, cansat-2022:Bno055, F.Cu at (180.8, 96.0)
- added U10: ~, Library:OKL, F.Cu at (190.5, 57.5)
- added U11: RASPBERRY_PI_4B_4GB, cansat-2022:raspberrypi, F.Cu at (63.5, 38.4)
- added U12: ~, Library:motor, F.Cu at (181.5, 96.4)
- added U2: BMP180, Connector_PinHeader_2.54mm:PinHeader_1x04_P2.54mm_Vertical, F.Cu at (180.0, 79.6)
- added U3: Lora, cansat-2022:LoRa, B.Cu at (202.4, 62.2)
- added U6: GPS, cansat-2022:GPS, F.Cu at (191.5, 41.5)
- added U9: MCP3002, Package_DIP:DIP-8_W7.62mm, B.Cu at (130.4, 40.0)
Routing:
- net GND: track 0.00 -> 518.5 mm, vias 0 -> 11
- net +3V3: track 0.00 -> 375.1 mm, vias 0 -> 3
- net +5V: track 0.00 -> 282.8 mm, vias 0 -> 2
- net VCC: track 0.00 -> 264.2 mm, vias 0 -> 7
- net /SDA: track 0.00 -> 258.4 mm, vias 0 -> 2
- net /SCL: track 0.00 -> 255.1 mm
- net +12V: track 0.00 -> 240.5 mm, vias 0 -> 5
- net Net-(J7-Pin_2): track 0.00 -> 168.5 mm, vias 0 -> 3
- net /ANALOG: track 0.00 -> 157.4 mm, vias 0 -> 3
- net /SEP_1: track 0.00 -> 146.0 mm, vias 0 -> 2
- net /GPS_TX: track 0.00 -> 143.4 mm, vias 0 -> 1
- net /TDF2_XSHUT: track 0.00 -> 143.4 mm
- net /GPS_RX: track 0.00 -> 142.7 mm, vias 0 -> 1
- net /LORA_TX: track 0.00 -> 140.0 mm
- net /PICO_RX: track 0.00 -> 137.2 mm
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- added copper zone on B.Cu, net GND
- added copper zone on F.Cu, net GND
Other:
- board outline added: 160 x 86 mm
- board text added: "Team Wolve'z 2026"
