File: mainboard2026_0522/mainboard2026_0522.kicad_pcb (KiCad board)
At the start: 2 copper layers, 160 x 86 mm, 41 parts, among them J1 Conn_01x06, J10 Conn_01x06_Pin, J11 Conn_01x02_Pin, J12 Conn_01x02_Pin, J13 Conn_01x02, J2 Conn_01x06, J3 Conn_01x02_Pin, J7 Conn_01x02, J8 Conn_01x03_Pin, J9 Conn_01x06_Pin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

Commit message: fix_pcb
Connections:
- 10k1 pad 2: VCC -> +3V3
- C1 pad 2: VCC -> +3V3
- C12 pad 2: VCC -> +3V3
- C13 pad 2: VCC -> +3V3
- C2 pad 1: VCC -> +3V3
- C3 pad 1: VCC -> +3V3
- J1 pad 3: VCC -> +3V3
- J2 pad 3: VCC -> +3V3
- R6 pad 2: VCC -> +3V3
- R9 pad 2: VCC -> +3V3
- U1 pad 1: VCC -> +3V3
- U2 pad 1: VCC -> +3V3
- U3 pad 13: VCC -> +3V3
- U3 pad 2: VCC -> +3V3
Routing:
- net +3V3: track 375.1 -> 670.9 mm, vias 3 -> 11
- net VCC: track 264.2 -> 0.00 mm, vias 7 -> 0
- net GND: vias 11 -> 12

Commit message: 2026_0528_19:50
Parts:
- added J4: Conn_01x06, Connector_JST:JST_ZH_S6B-ZR-SM4A-TF_1x06-1MP_P1.50mm_Horizontal, F.Cu at (77.2, 150.2)
- added J5: Conn_01x06, Connector_JST:JST_ZH_S6B-ZR-SM4A-TF_1x06-1MP_P1.50mm_Horizontal, F.Cu at (193.8, 150.7)
- added R10: 4.7k, Resistor_SMD:R_0603_1608Metric_Pad0.98x0.95mm_HandSolder, F.Cu at (157.5, 149.0)
- added R11: 4.7k, Resistor_SMD:R_0603_1608Metric_Pad0.98x0.95mm_HandSolder, F.Cu at (157.5, 151.5)
- added R14: 4.7k, Resistor_SMD:R_0603_1608Metric_Pad0.98x0.95mm_HandSolder, F.Cu at (157.5, 154.0)
- added R15: 4.7k, Resistor_SMD:R_0603_1608Metric_Pad0.98x0.95mm_HandSolder, F.Cu at (157.5, 156.5)

Commit message: wip
Parts:
- removed J10, J9: Conn_01x06_Pin, Connector_JST:JST_XH_S6B-XH-A-1_1x06_P2.50mm_Horizontal
- moved R15 38.4 mm to (165.6, 119.0)
- moved J5 32.7 mm to (195.5, 118.0), turned to 180 degrees
- moved J4 30.3 mm to (71.0, 120.5), turned to 180 degrees
- moved R10 13.1 mm to (148.4, 139.5)
Routing:
- net unconnected-(J5-Pin_6-Pad6): track 0.00 -> 125.3 mm
- net /SDA: track 258.4 -> 133.0 mm

Commit message: wip
Parts:
- J4, J5: moved to B.Cu
- moved J4 3.43 mm to (73.3, 118.0)
- moved J5 0.97 mm to (195.7, 119.0)
Routing:
- net unconnected-(J5-Pin_6-Pad6): track 125.3 -> 0.00 mm
- net /SDA: track 133.0 -> 258.4 mm
