File: mainboard2026_0522/mainboard2026_0522.kicad_pcb (KiCad board)
At the start: 2 copper layers, 160 x 86 mm, 43 parts, among them J1 Conn_01x06, J11 Conn_01x02_Pin, J12 Conn_01x02_Pin, J13 Conn_01x02, J2 Conn_01x06, J3 Conn_01x02_Pin, J4 Conn_01x06, J5 Conn_01x06, J7 Conn_01x02, J8 Conn_01x03_Pin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

Commit message: 20260601
Parts:
- moved R9 6.50 mm to (190.5, 91.0)
Changed lines of the file:
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@@
 		(capping no)
 		(filling no)
-		(zone_defaults)
 		(pcbplotparams
 			(layerselection 0x00000000_00000000_55555555_5755f5ff)
@@
 	(footprint "Resistor_SMD:R_0603_1608Metric_Pad0.98x0.95mm_HandSolder"
 		(layer "B.Cu")
-		(at 190.5 84.5 180)
+		(at 190.5 91 180)
 		(descr "Resistor SMD 0603 (1608 Metric), square (rectangular) end terminal, IPC-7351 nominal with elongated pad for handsoldering. (Body size source: IPC-SM-782 page 72, https://www.pcb-3d.com/wordpress/wp-content/uploads/ipc-sm-782a_amendment_1_and_2.pdf)")
 		(tags "resistor handsolder")
@@
 		(polygon
 			(pts
-				(xy 191.3125 85.45) (xy 191.5125 85.45) (xy 191.881921 84.828387) (xy 191.4125 84.499) (xy 190.943079 84.828387)
+				(xy 191.5125 90.05) (xy 191.3125 90.05) (xy 190.943079 90.671613) (xy 191.4125 91.001) (xy 191.881921 90.671613)
+			)
+		)
+	)
+	(zone
+		(net "Net-(J7-Pin_2)")
+		(layer "B.Cu")
+		(hatch none 0.1)
+		(priority 30094)
+		(attr
+			(teardrop
+				(type padvia)
+			)
+		)
+		(connect_pads yes
+			(clearance 0)
+		)
+		(min_thickness 0.0254)
+		(fill yes
+			(island_removal_mode 1)
+		)
+		(polygon
+			(pts
+				(xy 191.3125 91.95) (xy 191.5125 91.95) (xy 191.881921 91.328387) (xy 191.4125 90.999) (xy 190.943079 91.328387)
 			)
 		)
@@
 		(layer "B.Cu")
 		(hatch none 0.1)
-		(priority 30094)
+		(priority 30095)
 		(attr
 			(teardrop
@@
 	)
 	(zone
-		(net "+3V3")
-		(layer "B.Cu")
-		(hatch none 0.1)
-		(priority 30075)
-		(attr
-			(teardrop
-				(type padvia)
-			)
-		)
-		(connect_pads yes
-			(clearance 0)
-		)
-		(min_thickness 0.0254)
-		(fill yes
-			(island_removal_mode 1)
-		)
-		(polygon
-			(pts
-				(xy 189.8875 83.55) (xy 189.2875 83.55) (xy 189.118079 84.171613) (xy 189.5875 84.501) (xy 190.056921 84.171613)
-			)
-		)
-	)
-	(zone
 		(net "/GPS_TX")
 		(layer "B.Cu")
@@
 		(layer "B.Cu")
 		(hatch none 0.1)
+		(priority 30075)
+		(attr
+			(teardrop
+				(type padvia)
+			)
+		)
+		(connect_pads yes
+			(clearance 0)
+		)
+		(min_thickness 0.0254)
+		(fill yes
+			(island_removal_mode 1)
+		)
+		(polygon
+			(pts
+				(xy 189.8875 90.05) (xy 189.2875 90.05) (xy 189.118079 90.671613) (xy 189.5875 91.001) (xy 190.056921 90.671613)
+			)
+		)
+	)
+	(zone
+		(net "+3V3")
+		(layer "B.Cu")
+		(hatch none 0.1)
 		(priority 30076)
 		(attr
@@
 		(polygon
 			(pts
-				(xy 189.2875 85.45) (xy 189.8875 85.45) (xy 190.056921 84.828387) (xy 189.5875 84.499) (xy 189.118079 84.828387)
+				(xy 189.2875 91.95) (xy 189.8875 91.95) (xy 190.056921 91.328387) (xy 189.5875 90.999) (xy 189.118079 91.328387)
 			)
 		)
@@
 		(layer "B.Cu")
 		(hatch none 0.1)
-		(priority 30095)
+		(priority 30096)
 		(attr
 			(teardrop
@@
 		(layer "B.Cu")
 		(hatch none 0.1)
-		(priority 30096)
+		(priority 30097)
 		(attr
 			(teardrop
@@
 			)
 		)
-	)
-	(zone
-		(net "Net-(J7-Pin_2)")
-		(layer "B.Cu")
-		(hatch none 0.1)
-		(priority 30097)
-		(attr
-			(teardrop
-				(type padvia)
-			)
-		)
-		(connect_pads yes
-			(clearance 0)
-		)
-		(min_thickness 0.0254)
-		(fill yes
-			(island_removal_mode 1)
-		)
-		(polygon
-			(pts
-				(xy 191.5125 83.55) (xy 191.3125 83.55) (xy 190.943079 84.171613) (xy 191.4125 84.501) (xy 191.881921 84.171613)
-			)
-		)

Commit message: fix
Routing:
- net GND: vias 29 -> 34
