File: mainboard2026_0522/mainboard2026_0522.kicad_pcb (KiCad board)
At the start: 2 copper layers, 160 x 86 mm, 43 parts, among them J1 Conn_01x06, J11 Conn_01x02_Pin, J12 Conn_01x02_Pin, J13 Conn_01x02, J2 Conn_01x06, J3 Conn_01x02_Pin, J4 Conn_01x06, J5 Conn_01x06, J7 Conn_01x02, J8 Conn_01x03_Pin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

Commit message: ver1complete
Parts:
- J11: moved to F.Cu

Commit message: fixpcb
Connections:
- U11 pad 12: /LORA_TX -> unconnected-(U11-GPIO18/GPIO_GEN1-Pad12)
- U11 pad 13: /LORA_RX -> Net-(J7-Pin_2)
- U11 pad 29: unconnected-(U11-GPIO5-Pad29) -> /LORA_TX
- U11 pad 7: Net-(J7-Pin_2) -> /LORA_RX
Routing:
- net /LORA_TX: track 155.9 -> 149.3 mm, vias 0 -> 2
- net Net-(J7-Pin_2): track 167.1 -> 163.9 mm
- net /LORA_RX: track 152.6 -> 154.1 mm, vias 0 -> 2
- net /SW: track 115.0 -> 116.4 mm
