File: mainboard2026_0522/mainboard2026_0522.kicad_pcb (KiCad board)
At the start: 2 copper layers, 160 x 86 mm, 43 parts, among them J1 Conn_01x06, J11 Conn_01x02_Pin, J12 Conn_01x02_Pin, J13 Conn_01x02, J2 Conn_01x06, J3 Conn_01x02_Pin, J4 Conn_01x06, J5 Conn_01x06, J7 Conn_01x02, J8 Conn_01x03_Pin, Q1 Q_NMOS_GDS, Q2 Q_NMOS_GDS, SW1 SW_SPDT, SW2 SW_Push, U1 Bno055, U11 RASPBERRY_PI_4B_4GB, U2 BMP180, U3 Lora, U6 GPS, U9 MCP3002

Commit message: add logo
Parts:
- added G***: LOGO, LOGO, F.Cu at (135.0, 113.5)
Other:
- board text added: "Wolve'Z 2026"
- board text removed: "Team Wolve'z 2026"

Commit message: board fix
Parts:
- added Q3: Q_NMOS_GDS, Package_TO_SOT_SMD:TO-252-3_TabPin2, F.Cu at (199.0, 68.5)
- added R7: 100k, Resistor_SMD:R_0603_1608Metric_Pad0.98x0.95mm_HandSolder, F.Cu at (191.5, 70.0)
- added SW3: SW_SPDT, Button_Switch_THT:SW_Slide-03_Wuerth-WS-SLTV_10x2.5x6.4_P2.54mm, F.Cu at (205.5, 71.5)
- R4, R5: footprint Resistor_SMD:R_0603_1608Metric_Pad0.98x0.95mm_HandSolder -> Resistor_THT:R_Axial_DIN0207_L6.3mm_D2.5mm_P10.16mm_Horizontal
- moved R4 73.7 mm to (178.7, 104.5)
- moved R5 3.67 mm to (192.1, 101.0)
- moved U2 1.42 mm to (186.5, 73.1)
Connections:
- U10 pad 2: GND -> Net-(Q3-D)
- U11 pad 6: (no net) -> GND
Routing:
- net Net-(Q3-G): track 0.00 -> 20.4 mm
- net Net-(Q3-D): track 0.00 -> 16.0 mm
- net GND: track 584.5 -> 600.1 mm, vias 34 -> 33
- net /SCL: track 247.0 -> 256.9 mm, vias 1 -> 3
- net Net-(J3-Pin_1): track 18.7 -> 13.6 mm, vias 1 -> 0
- net +12V: track 108.5 -> 112.4 mm
- net Net-(J12-Pin_1): track 19.1 -> 22.3 mm
- net /SDA: track 267.9 -> 269.3 mm
- net Net-(J11-Pin_1): track 31.3 -> 32.1 mm
Other:
- outline, holes or cut-outs redrawn
- board text added: "+ in"
- board text added: "- in"
