File: mainboard2026_0522/mainboard2026_0522.kicad_sch (KiCad schematic)
At the start: 45 parts, among them J1 Conn_01x06, J11 Conn_01x02_Pin, J12 Conn_01x02_Pin, J13 Conn_01x02, J2 Conn_01x06, J3 Conn_01x02_Pin, J4 Conn_01x06, J5 Conn_01x06, J7 Conn_01x02, J8 Conn_01x03_Pin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

Commit message: wip
Parts:
- J4, J5: footprint Connector_JST:JST_ZH_S6B-ZR-SM4A-TF_1x06-1MP_P1.50mm_Horizontal -> CANSAT2026:JST_ZH_B6B-ZR_1x06_P1.50mm_Horizontal
Changed lines of the file:
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@@
 			)
 		)
-		(property "Footprint" "Connector_JST:JST_ZH_S6B-ZR-SM4A-TF_1x06-1MP_P1.50mm_Horizontal"
+		(property "Footprint" "CANSAT2026:JST_ZH_B6B-ZR_1x06_P1.50mm_Horizontal"
 			(at 330.2 125.73 0)
 			(hide yes)
@@
 			)
 		)
-		(property "Footprint" "Connector_JST:JST_ZH_S6B-ZR-SM4A-TF_1x06-1MP_P1.50mm_Horizontal"
+		(property "Footprint" "CANSAT2026:JST_ZH_B6B-ZR_1x06_P1.50mm_Horizontal"
 			(at 330.2 151.13 0)
 			(hide yes)
