File: mainboard2026_0522/mainboard2026_0522.kicad_sch (KiCad schematic)
At the start: 43 parts, among them J1 Conn_01x06, J10 Conn_01x06_Pin, J11 Conn_01x02_Pin, J12 Conn_01x02_Pin, J2 Conn_01x06, J3 Conn_01x02_Pin, J5 Conn_01x02, J6 Conn_01x02, J7 Conn_01x02, J8 Conn_01x03_Pin, J9 Conn_01x06_Pin, Q1 Q_NMOS_GDS, Q2 Q_NMOS_GDS, SW1 SW_SPDT, SW2 SW_Push, U1 Bno055, U11 RASPBERRY_PI_4B_4GB, U2 BMP180, U3 Lora, U6 GPS, U8 CH340N, U9 MCP3002

Commit message: schfinished
Parts:
- U11: footprint Module:Raspberry_Pi_Zero_Socketed_THT_FaceDown_MountingHoles -> CANSAT2026:RaspberryPi_4B_40pin_Mount
- U12, U7: value ~ -> (none)
Connections:
- net GND: no longer U11.6 (GND), U11.S1 (SHIELD), U11.S2 (SHIELD__1), U11.S3 (SHIELD__2), U11.S4 (SHIELD__3)
- no-connect marks 50 -> 46

Commit message: 20260524
Parts:
- removed U7: (no value), Library:OKL, symbol Library:XL4015
- added J13: Conn_01x02, Connector_AMASS:AMASS_XT30U-M_1x02_P5.0mm_Vertical, symbol Connector_Generic:Conn_01x02
- added U10: ~, Library:OKL, symbol Library:XL4015
- J5: footprint CANSAT2026:BT_connecta -> Connector_JST:JST_PH_B2B-PH-K_1x02_P2.00mm_Vertical
Connections:
- net +12V: now also J13.2 (Pin_2), U10.1 (IN+)
- net +5V: now also U10.3 (OUT+)
- net GND: now also J13.1 (Pin_1), U10.2 (IN-), U10.4 (OUT-)
- no-connect marks 46 -> 45

Commit message: 2026_0524_19:07
Parts:
- removed C7: 0.1u, Capacitor_SMD:C_0603_1608Metric_Pad1.08x0.95mm_HandSolder, symbol Device:C
- removed J6: Conn_01x02, Connector_JST:JST_PH_B2B-PH-K_1x02_P2.00mm_Vertical, symbol Connector_Generic:Conn_01x02
- removed U8: CH340N, Package_SO:SOIC-8_3.9x4.9mm_P1.27mm, symbol Interface_USB:CH340N
- R12, R2: value R -> 10k
Connections:
- net LORA_RX: now also U11.13 (GPIO27/GPIO_GEN2)
- net LORA_TX: now also U11.12 (GPIO18/GPIO_GEN1)
- net RESET: now also U11.16 (GPIO23/GPIO_GEN4); no longer U11.12 (GPIO18/GPIO_GEN1)
- no-connect marks 45 -> 42

Commit message: pcb_precomplete
Parts:
- removed J5: Conn_01x02, Connector_JST:JST_PH_B2B-PH-K_1x02_P2.00mm_Vertical, symbol Connector_Generic:Conn_01x02
- added C11: 0.1u, Capacitor_SMD:C_0603_1608Metric_Pad1.08x0.95mm_HandSolder, symbol Device:C
- J8: footprint Connector:FanPinHeader_1x03_P2.54mm_Vertical -> Connector_JST:JST_PH_B3B-PH-K_1x03_P2.00mm_Vertical
- U11: footprint CANSAT2026:RaspberryPi_4B_40pin_Mount -> cansat-2022:raspberrypi
Connections:
- net 3V3 is gone; now on net +3V3: R5.1, U11.1 (3V3), U11.17 (3V3__1), U9.8 (VDD/VREF)
- net +3V3: now also C11.1
- net GND: now also C11.2

Commit message: fix_pcb
Connections:
- net VCC is gone; now on net +3V3: 10k1.2, C1.2, C12.2, C13.2, C2.1, C3.1, J1.3 (Pin_3), J2.3 (Pin_3), R6.2, R9.2, U1.1 (Vin), U2.1 (VIN), U3.13 (Vcc), U3.2 (VccRF)
Changed lines of the file:
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@@
 	)
 	(junction
-		(at 208.28 91.44)
+		(at 209.55 88.9)
 		(diameter 0)
 		(color 0 0 0 0)
 	)
 	(junction
-		(at 135.89 242.57)
+		(at 208.28 91.44)
 		(diameter 0)
 		(color 0 0 0 0)
 	)
 	(junction
-		(at 46.355 129.54)
+		(at 135.89 242.57)
 		(diameter 0)
 		(color 0 0 0 0)
 	)
 	(junction
-		(at 326.39 176.53)
+		(at 46.355 129.54)
 		(diameter 0)
 		(color 0 0 0 0)
 	)
 	(junction
-		(at 391.16 78.74)
+		(at 326.39 176.53)
 		(diameter 0)
 		(color 0 0 0 0)
@@
 	(wire
 		(pts
-			(xy 208.28 88.9) (xy 210.82 88.9)
+			(xy 208.28 88.9) (xy 209.55 88.9)
 		)
 		(stroke
@@
 	(wire
 		(pts
+			(xy 209.55 87.63) (xy 209.55 88.9)
+		)
+		(stroke
+			(width 0)
+			(type default)
+		)
+	)
+	(wire
+		(pts
 			(xy 29.21 85.09) (xy 34.29 85.09)
 		)
@@
 	(wire
 		(pts
+			(xy 212.09 87.63) (xy 209.55 87.63)
+		)
+		(stroke
+			(width 0)
+			(type default)
+		)
+	)
+	(wire
+		(pts
 			(xy 53.34 76.2) (xy 53.34 80.01)
 		)
@@
 	(wire
 		(pts
-			(xy 386.08 87.63) (xy 386.08 92.71)
+			(xy 214.63 86.36) (xy 212.09 86.36)
 		)
 		(stroke
@@
 	(wire
 		(pts
-			(xy 144.78 129.54) (xy 154.94 129.54)
+			(xy 386.08 87.63) (xy 386.08 92.71)
 		)
 		(stroke
@@
 	(wire
 		(pts
-			(xy 392.43 78.74) (xy 391.16 78.74)
+			(xy 144.78 129.54) (xy 154.94 129.54)
 		)
 		(stroke
@@
 	(wire
 		(pts
-			(xy 331.47 85.09) (xy 331.47 78.74)
+			(xy 389.89 78.74) (xy 392.43 78.74)
 		)
 		(stroke
@@
 	(wire
 		(pts
-			(xy 321.31 152.4) (xy 337.82 152.4)
+			(xy 331.47 85.09) (xy 331.47 78.74)
 		)
 		(stroke
@@
 	(wire
 		(pts
-			(xy 337.82 182.88) (xy 340.36 182.88)
+			(xy 321.31 152.4) (xy 337.82 152.4)
 		)
 		(stroke
@@
 	(wire
 		(pts
-			(xy 144.78 99.06) (xy 154.94 99.06)
+			(xy 337.82 182.88) (xy 340.36 182.88)
 		)
 		(stroke
@@
 	(wire
 		(pts
-			(xy 144.78 114.3) (xy 154.94 114.3)
+			(xy 144.78 99.06) (xy 154.94 99.06)
 		)
 		(stroke
@@
 	(wire
 		(pts
-			(xy 120.65 111.76) (xy 125.73 111.76)
+			(xy 144.78 114.3) (xy 154.94 114.3)
 		)
 		(stroke
@@
 	(wire
 		(pts
-			(xy 391.16 78.74) (xy 389.89 78.74)
+			(xy 120.65 111.76) (xy 125.73 111.76)
 		)
 		(stroke
@@
 	(wire
 		(pts
+			(xy 209.55 88.9) (xy 210.82 88.9)
+		)
+		(stroke
+			(width 0)
+			(type default)
+		)
+	)
+	(wire
+		(pts
 			(xy 382.27 87.63) (xy 386.08 87.63)
 		)
@@
 		)
 	)
+	(wire
+		(pts
+			(xy 212.09 86.36) (xy 212.09 87.63)
+		)
+		(stroke
+			(width 0)
+			(type default)
+		)
+	)
 	(label "SPI0_MOSI"
 		(at 144.78 127 0)
@@
 	)
 	(symbol
+		(lib_name "VCC_1")
+		(lib_id "power:VCC")
+		(at 214.63 86.36 0)
+		(unit 1)
+		(body_style 1)
+		(exclude_from_sim no)
+		(in_bom yes)
+		(on_board yes)
+		(in_pos_files yes)
+		(dnp no)
+		(fields_autoplaced yes)
+		(property "Reference" "#PWR040"
+			(at 214.63 90.17 0)
+			(hide yes)
+			(show_name no)
+			(do_not_autoplace no)
+			(effects
+				(font
+					(size 1.27 1.27)
+				)
+			)
+		)
+		(property "Value" "VCC"
+			(at 214.63 81.28 0)
+			(show_name no)
+			(do_not_autoplace no)
+			(effects
+				(font
+					(size 1.27 1.27)
+				)
+			)
+		)
+		(property "Footprint" ""
+			(at 214.63 86.36 0)
+			(hide yes)
+			(show_name no)
+			(do_not_autoplace no)
+			(effects
+				(font
+					(size 1.27 1.27)
+				)
+			)
+		)
+		(property "Datasheet" ""
+			(at 214.63 86.36 0)
+			(hide yes)
+			(show_name no)
+			(do_not_autoplace no)
+			(effects
+				(font
+					(size 1.27 1.27)
+				)
+			)
+		)
+		(property "Description" "Power symbol creates a global label with name \"VCC\""
+			(at 214.63 86.36 0)
+			(hide yes)
+			(show_name no)
+			(do_not_autoplace no)
+			(effects
+				(font
+					(size 1.27 1.27)
+				)
+			)
+		)
+		(pin "1"
+		)
+		(instances
+			(project "mainboard2026_0522"
+				(path "/1476b0f4-e0d9-4b9a-b2f2-db212dad2049"
+					(reference "#PWR040")
+					(unit 1)
+				)
+			)
+		)
+	)
+	(symbol
 		(lib_id "RASPBERRY_PI_4B_4GB:RASPBERRY_PI_4B_4GB")
 		(at 180.34 114.3 0)
@@
 					(unit 1)
 				)
-			)
-		)
-	)
-	(symbol
-		(lib_id "power:PWR_FLAG")
-		(at 391.16 78.74 180)
-		(unit 1)
-		(body_style 1)
-		(exclude_from_sim no)
-		(in_bom yes)
-		(on_board yes)
-		(in_pos_files yes)
-		(dnp no)
-		(fields_autoplaced yes)
-		(property "Reference" "#FLG01"
-			(at 391.16 80.645 0)
-			(hide yes)
-			(show_name no)
-			(do_not_autoplace no)
-			(effects
-				(font
-					(size 1.27 1.27)
-				)
-			)
-		)
-		(property "Value" "PWR_FLAG"
-			(at 391.16 83.82 0)
-			(show_name no)
-			(do_not_autoplace no)
-			(effects
-				(font
-					(size 1.27 1.27)
-				)
-			)
-		)
-		(property "Footprint" ""
-			(at 391.16 78.74 0)
-			(hide yes)
-			(show_name no)
-			(do_not_autoplace no)
-			(effects
-				(font
-					(size 1.27 1.27)
-				)
-			)
-		)
-		(property "Datasheet" ""
-			(at 391.16 78.74 0)
-			(hide yes)
-			(show_name no)
-			(do_not_autoplace no)
-			(effects
-				(font
-					(size 1.27 1.27)
-				)
-			)
-		)
-		(property "Description" "Special symbol for telling ERC where power comes from"
-			(at 391.16 78.74 0)
-			(hide yes)
-			(show_name no)
-			(do_not_autoplace no)
-			(effects
-				(font
-					(size 1.27 1.27)
-				)
-			)
-		)
-		(pin "1"
-		)
-		(instances
-			(project "mainboard2026_0522"
-				(path "/1476b0f4-e0d9-4b9a-b2f2-db212dad2049"
-					(reference "#FLG01")
-					(unit 1)
-				)

Commit message: 2026_0528_19:50
Parts:
- removed J10, J9: Conn_01x06_Pin, Connector_JST:JST_XH_S6B-XH-A-1_1x06_P2.50mm_Horizontal, symbol Connector:Conn_01x06_Pin
- added J4, J5: Conn_01x06, Connector_JST:JST_ZH_S6B-ZR-SM4A-TF_1x06-1MP_P1.50mm_Horizontal, symbol Connector_Generic:Conn_01x06
- added R10, R11, R14, R15: 4.7k, Resistor_SMD:R_0603_1608Metric_Pad0.98x0.95mm_HandSolder, symbol Device:R
Connections:
- net +3V3: now also J4.1 (Pin_1), J5.1 (Pin_1), R10.2, R11.2, R14.2, R15.2
- net GND: now also J4.2 (Pin_2), J5.2 (Pin_2)
- net SCL: now also J4.4 (Pin_4), J5.4 (Pin_4), R11.1, R14.1
- net SDA: now also J4.3 (Pin_3), J5.3 (Pin_3), R10.1, R15.1
- net TDF1_XSHUT: now also J4.5 (Pin_5), J5.5 (Pin_5)
- no-connect marks 42 -> 41

Commit message: wip
Connections:
- net GND: now also U9.2 (CH0)
- no-connect marks 41 -> 40
Changed lines of the file:
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@@
 	)
 	(no_connect
-		(at 204.47 224.79)
-	)
-	(no_connect
 		(at 311.15 133.35)
 	)
@@
 	(wire
 		(pts
-			(xy 204.47 224.79) (xy 217.17 224.79)
-		)
-		(stroke
-			(width 0)
-			(type default)
-		)
-	)
-	(wire
-		(pts
 			(xy 144.78 124.46) (xy 154.94 124.46)
 		)
@@
 	(wire
 		(pts
+			(xy 209.55 224.79) (xy 217.17 224.79)
+		)
+		(stroke
+			(width 0)
+			(type default)
+		)
+	)
+	(wire
+		(pts
 			(xy 229.87 213.36) (xy 229.87 217.17)
 		)
@@
 					(unit 1)
 				)
+			)
+		)
+	)
+	(symbol
+		(lib_name "GND_4")
+		(lib_id "power:GND")
+		(at 209.55 224.79 0)
+		(unit 1)
+		(body_style 1)
+		(exclude_from_sim no)
+		(in_bom yes)
+		(on_board yes)
+		(in_pos_files yes)
+		(dnp no)
+		(fields_autoplaced yes)
+		(property "Reference" "#PWR048"
+			(at 209.55 231.14 0)
+			(hide yes)
+			(show_name no)
+			(do_not_autoplace no)
+			(effects
+				(font
+					(size 1.27 1.27)
+				)
+			)
+		)
+		(property "Value" "GND"
+			(at 209.55 229.87 0)
+			(show_name no)
+			(do_not_autoplace no)
+			(effects
+				(font
+					(size 1.27 1.27)
+				)
+			)
+		)
+		(property "Footprint" ""
+			(at 209.55 224.79 0)
+			(hide yes)
+			(show_name no)
+			(do_not_autoplace no)
+			(effects
+				(font
+					(size 1.27 1.27)
+				)
+			)
+		)
+		(property "Datasheet" ""
+			(at 209.55 224.79 0)
+			(hide yes)
+			(show_name no)
+			(do_not_autoplace no)
+			(effects
+				(font
+					(size 1.27 1.27)
+				)
+			)
+		)
+		(property "Description" "Power symbol creates a global label with name \"GND\" , ground"
+			(at 209.55 224.79 0)
+			(hide yes)
+			(show_name no)
+			(do_not_autoplace no)
+			(effects
+				(font
+					(size 1.27 1.27)
+				)
+			)
+		)
+		(pin "1"
+		)
+		(instances
+			(project "mainboard2026_0522"
+				(path "/1476b0f4-e0d9-4b9a-b2f2-db212dad2049"
+					(reference "#PWR048")
+					(unit 1)
+				)

Commit message: pcb0529
Parts:
- removed R14, R15: 4.7k, Resistor_SMD:R_0603_1608Metric_Pad0.98x0.95mm_HandSolder, symbol Device:R
- J4, J5: footprint Connector_JST:JST_ZH_S6B-ZR-SM4A-TF_1x06-1MP_P1.50mm_Horizontal -> CANSAT2026:JST_ZH_B6B-ZR_1x06_P1.50mm_Horizontal
Connections:
- net TDF1_XSHUT: no longer J5.5 (Pin_5)
- net TDF2_XSHUT: now also J5.5 (Pin_5)
Changed lines of the file:
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@@
 	)
 	(junction
-		(at 298.45 146.05)
-		(diameter 0)
-		(color 0 0 0 0)
-	)
-	(junction
 		(at 205.74 165.1)
 		(diameter 0)
@@
 	)
 	(junction
-		(at 290.83 146.05)
-		(diameter 0)
-		(color 0 0 0 0)
-	)
-	(junction
 		(at 123.19 245.11)
 		(diameter 0)
@@
 	(wire
 		(pts
-			(xy 298.45 146.05) (xy 298.45 151.13)
-		)
-		(stroke
-			(width 0)
-			(type default)
-		)
-	)
-	(wire
-		(pts
-			(xy 290.83 146.05) (xy 290.83 153.67)
-		)
-		(stroke
-			(width 0)
-			(type default)
-		)
-	)
-	(wire
-		(pts
 			(xy 134.62 96.52) (xy 138.43 96.52)
 		)
@@
 	(wire
 		(pts
-			(xy 311.15 156.21) (xy 325.12 156.21)
+			(xy 307.34 156.21) (xy 325.12 156.21)
 		)
 		(stroke
@@
 	(wire
 		(pts
-			(xy 287.02 146.05) (xy 290.83 146.05)
-		)
-		(stroke
-			(width 0)
-			(type default)
-		)
-	)
-	(wire
-		(pts
 			(xy 144.78 127) (xy 154.94 127)
 		)
@@
 	(wire
 		(pts
-			(xy 298.45 146.05) (xy 325.12 146.05)
-		)
-		(stroke
-			(width 0)
-			(type default)
-		)
-	)
-	(wire
-		(pts
 			(xy 204.47 234.95) (xy 217.17 234.95)
 		)
@@
 	(wire
 		(pts
-			(xy 290.83 146.05) (xy 298.45 146.05)
+			(xy 287.02 146.05) (xy 325.12 146.05)
 		)
 		(stroke
@@
 		)
 	)
-	(label "TDF1_XSHUT"
-		(at 311.15 156.21 180)
+	(label "TDF2_XSHUT"
+		(at 307.34 156.21 180)
 		(effects
 			(font
@@
 			)
 		)
-		(property "Footprint" "Connector_JST:JST_ZH_S6B-ZR-SM4A-TF_1x06-1MP_P1.50mm_Horizontal"
+		(property "Footprint" "CANSAT2026:JST_ZH_B6B-ZR_1x06_P1.50mm_Horizontal"
 			(at 330.2 125.73 0)
 			(hide yes)
@@
 	)
 	(symbol
-		(lib_id "Device:R")
-		(at 302.26 151.13 270)
-		(unit 1)
-		(body_style 1)
-		(exclude_from_sim no)
-		(in_bom yes)
-		(on_board yes)
-		(in_pos_files yes)
-		(dnp no)
-		(fields_autoplaced yes)
-		(property "Reference" "R15"
-			(at 302.26 144.78 90)
-			(show_name no)
-			(do_not_autoplace no)
-			(effects
-				(font
-					(size 1.27 1.27)
-				)
-			)
-		)
-		(property "Value" "4.7k"
-			(at 302.26 147.32 90)
-			(show_name no)
-			(do_not_autoplace no)
-			(effects
-				(font
-					(size 1.27 1.27)
-				)
-			)
-		)
-		(property "Footprint" "Resistor_SMD:R_0603_1608Metric_Pad0.98x0.95mm_HandSolder"
-			(at 302.26 149.352 90)
-			(hide yes)
-			(show_name no)
-			(do_not_autoplace no)
-			(effects
-				(font
-					(size 1.27 1.27)
-				)
-			)
-		)
-		(property "Datasheet" ""
-			(at 302.26 151.13 0)
-			(hide yes)
-			(show_name no)
-			(do_not_autoplace no)
-			(effects
-				(font
-					(size 1.27 1.27)
-				)
-			)
-		)
-		(property "Description" ""
-			(at 302.26 151.13 0)
-			(hide yes)
-			(show_name no)
-			(do_not_autoplace no)
-			(effects
-				(font
-					(size 1.27 1.27)
-				)
-			)
-		)
-		(pin "1"
-		)
-		(pin "2"
-		)
-		(instances
-			(project "mainboard2026_0522"
-				(path "/1476b0f4-e0d9-4b9a-b2f2-db212dad2049"
-					(reference "R15")
-					(unit 1)
-				)
-			)
-		)
-	)
-	(symbol
 		(lib_id "Library:XL4015")
 		(at 146.05 243.84 0)
@@
 			)
 		)
-		(property "Footprint" "Connector_JST:JST_ZH_S6B-ZR-SM4A-TF_1x06-1MP_P1.50mm_Horizontal"
+		(property "Footprint" "CANSAT2026:JST_ZH_B6B-ZR_1x06_P1.50mm_Horizontal"
 			(at 330.2 151.13 0)
 			(hide yes)
@@
 					(unit 1)
 				)
-			)
-		)
-	)
-	(symbol
-		(lib_id "Device:R")
-		(at 294.64 153.67 270)
-		(unit 1)
-		(body_style 1)
-		(exclude_from_sim no)
-		(in_bom yes)
-		(on_board yes)
-		(in_pos_files yes)
-		(dnp no)
-		(fields_autoplaced yes)
-		(property "Reference" "R14"
-			(at 294.64 147.32 90)
-			(show_name no)
-			(do_not_autoplace no)
-			(effects
-				(font
-					(size 1.27 1.27)
-				)
-			)
-		)
-		(property "Value" "4.7k"
-			(at 294.64 149.86 90)
-			(show_name no)
-			(do_not_autoplace no)
-			(effects
-				(font
-					(size 1.27 1.27)
-				)
-			)
-		)
-		(property "Footprint" "Resistor_SMD:R_0603_1608Metric_Pad0.98x0.95mm_HandSolder"
-			(at 294.64 151.892 90)
-			(hide yes)
-			(show_name no)
-			(do_not_autoplace no)
-			(effects
-				(font
-					(size 1.27 1.27)
-				)
-			)
-		)
-		(property "Datasheet" ""
-			(at 294.64 153.67 0)
-			(hide yes)
-			(show_name no)
-			(do_not_autoplace no)
-			(effects
-				(font
-					(size 1.27 1.27)
-				)
-			)
-		)
-		(property "Description" ""
-			(at 294.64 153.67 0)
-			(hide yes)
-			(show_name no)
-			(do_not_autoplace no)
-			(effects
-				(font
-					(size 1.27 1.27)
-				)
-			)
-		)
-		(pin "1"
-		)
-		(pin "2"
-		)
-		(instances
-			(project "mainboard2026_0522"
-				(path "/1476b0f4-e0d9-4b9a-b2f2-db212dad2049"
-					(reference "R14")
-					(unit 1)
-				)
