File: mainboard2026_0522/mainboard2026_0522.kicad_sch (KiCad schematic)
At the start: 43 parts, among them J1 Conn_01x06, J11 Conn_01x02_Pin, J12 Conn_01x02_Pin, J13 Conn_01x02, J2 Conn_01x06, J3 Conn_01x02_Pin, J4 Conn_01x06, J5 Conn_01x06, J7 Conn_01x02, J8 Conn_01x03_Pin, Q1 Q_NMOS_GDS, Q2 Q_NMOS_GDS, SW1 SW_SPDT, SW2 SW_Push, U1 Bno055, U11 RASPBERRY_PI_4B_4GB, U2 BMP180, U3 Lora, U6 GPS, U9 MCP3002

Commit message: board fix
Parts:
- added Q3: Q_NMOS_GDS, Package_TO_SOT_SMD:TO-252-3_TabPin2, symbol Device:Q_NMOS_GDS
- added R7: 100k, Resistor_SMD:R_0603_1608Metric_Pad0.98x0.95mm_HandSolder, symbol Device:R
- added SW3: SW_SPDT, Button_Switch_THT:SW_Slide-03_Wuerth-WS-SLTV_10x2.5x6.4_P2.54mm, symbol Switch:SW_SPDT
- R4, R5: footprint Resistor_SMD:R_0603_1608Metric_Pad0.98x0.95mm_HandSolder -> Resistor_THT:R_Axial_DIN0207_L6.3mm_D2.5mm_P10.16mm_Horizontal
Connections:
- net +12V: now also SW3.2 (B)
- net GND: now also U11.6 (GND__8), Q3.3 (S), R7.1; no longer U10.2 (IN-)
- new net: Q3.2 (D), U10.2 (IN-)
- new net: Q3.1 (G), R7.2, SW3.1 (A)
- no-connect marks 40 -> 41
Other:
- moved on the sheet: J13
